File: driver_bts7960_v2_industrial/driver_bts7960_v2_industrial.kicad_pcb (KiCad board)
At the start: 2 copper layers, 50.3 x 45 mm, 32 parts, among them J1 Motor_1, J2 XT30, J3 Conn_01x08_Pin, J6 Motor_2, U1 BTS7960B, U2 BTS7960B, U3 BTS7960B, U4 BTS7960B, U5 74HC244

Commit message: .
Parts:
- J1: value Motor_1 -> XT30
- J3: value Conn_01x08_Pin -> Pin Header M 01x08
- J6: value Motor_2 -> XT30
- R1, R10, R2, R3, R4, R5, R6, R7, R8, R9: value 10k -> 10k 0805
- R11, R12, R13, R14: value 30k -> 30k 0805
- moved C4 0.59 mm to (156.8, 59.1)
Routing:
- net Net-(J6-Pin_2): track 13.8 -> 37.3 mm, vias 9 -> 43
- net Net-(J1-Pin_2): track 8.66 -> 26.6 mm, vias 9 -> 43
- net Net-(J1-Pin_1): track 24.3 -> 38.9 mm, vias 9 -> 42
- net Net-(J6-Pin_1): track 15.0 -> 24.0 mm, vias 9 -> 42
- net GND: track 198.9 -> 197.8 mm
- net OUT_EN_2: track 42.5 -> 43.6 mm
- net VS: track 75.8 -> 76.8 mm
- net Net-(U3-IS): track 20.4 -> 21.3 mm
